Commit message: backup aula 15

File: description/camera.xacro (robot description, xacro)
@@ -4,5 +4,5 @@
         <parent link="chassis"/>
         <child link="camera_link"/>
-        <origin xyz="0.276 0 0.181" rpy="0 0 0"/>
+        <origin xyz="0.4 0 0.30" rpy="0 0 0"/>
     </joint>
     <link name="camera_link">

File: description/depth_camera.xacro (robot description, xacro)
@@ -4,5 +4,5 @@
         <parent link="chassis"/>
         <child link="camera_link"/>
-        <origin xyz="0.305 0 0.08" rpy="0 0 0"/>
+        <origin xyz="0.47 0 0.1" rpy="0 0 0"/>
     </joint>
     <link name="camera_link">

File: description/lidar.xacro (robot description, xacro)
@@ -4,5 +4,5 @@
         <parent link="chassis"/>
         <child link="laser_frame"/>
-        <origin xyz="0.122 0 0.212" rpy="0 0 0"/>
+        <origin xyz="0.122 0 0.300" rpy="0 0 0"/>
     </joint>
     <link name="laser_frame">

File: description/robot_core.xacro (robot description, xacro)
@@ -2,17 +2,17 @@
 <robot xmlns:xacro="http://www.ros.org/wiki/xacro" >
     <xacro:include filename="inertial_macros.xacro"/>
-    <xacro:property name="chassis_length" value="0.335"/>
-    <xacro:property name="chassis_width" value="0.265"/>
-    <xacro:property name="chassis_height" value="0.138"/>
-    <xacro:property name="chassis_mass" value="1.0"/>
-    <xacro:property name="wheel_radius" value="0.033"/>
-    <xacro:property name="wheel_thickness" value="0.026"/>
-    <xacro:property name="wheel_mass" value="0.05"/>
-    <xacro:property name="wheel_offset_x" value="0.226"/>
-    <xacro:property name="wheel_offset_y" value="0.1485"/>
-    <xacro:property name="wheel_offset_z" value="0.01"/>
-    <xacro:property name="caster_wheel_radius" value="0.01"/>
-    <xacro:property name="caster_wheel_mass" value="0.01"/>
-    <xacro:property name="caster_wheel_offset_x" value="0.075"/>
+    <xacro:property name="chassis_length" value="0.4661"/>
+    <xacro:property name="chassis_width" value="0.384"/>
+    <xacro:property name="chassis_height" value="0.276"/>
+    <xacro:property name="chassis_mass" value="5.75"/>
+    <xacro:property name="wheel_radius" value="0.042"/>
+    <xacro:property name="wheel_thickness" value="0.04"/>
+    <xacro:property name="wheel_mass" value="0.072"/>
+    <xacro:property name="wheel_offset_x" value="0.341"/>
+    <xacro:property name="wheel_offset_y" value="0.217"/>
+    <xacro:property name="wheel_offset_z" value="-0.02"/>
+    <xacro:property name="caster_wheel_radius" value="0.025"/>
+    <xacro:property name="caster_wheel_mass" value="0.05"/>
+    <xacro:property name="caster_wheel_offset_x" value="0.115"/>
     <xacro:property name="caster_wheel_offset_z" value="${wheel_offset_z - wheel_radius + caster_wheel_radius}"/>
     <material name="white">

File: description/ros2_control.xacro (robot description, xacro)
@@ -11,5 +11,6 @@
                 <param name="baud_rate">57600</param>
                 <param name="timeout">1000</param>
-                <param name="enc_counts_per_rev">3436</param>
+                <!--<param name="enc_counts_per_rev">3436</param> -->
+                <param name="enc_counts_per_rev">440</param>
             </hardware>
             <joint name="left_wheel_joint">
